File: comfrey77_PCB/comfrey77.sch (KiCad schematic (older format))
At the start: 249 parts, among them J1 Conn_01x02, J10 Conn_01x01, J11 Conn_01x01, J12 Conn_01x01, J13 Conn_01x01, J14 Conn_01x01, J15 Conn_01x01, J16 Conn_01x01, J17 Conn_01x01, J2 Conn_01x01, J3 Conn_01x01, J4 Conn_01x01, J5 Conn_01x01, J6 Conn_01x01, J7 Conn_01x01, J8 Conn_01x01, J9 Conn_01x01, SW1 SW_PUSH, SW10 SW_PUSH, SW11 SW_PUSH, SW12 SW_PUSH, SW13 SW_PUSH, SW14 SW_PUSH, SW15 SW_PUSH, SW16 SW_PUSH, SW17 SW_PUSH, SW18 SW_PUSH, SW19 SW_PUSH, SW2 SW_PUSH, SW20 SW_PUSH, SW21 SW_PUSH, SW22 SW_PUSH, SW23 SW_PUSH, SW24 SW_PUSH, SW25 SW_PUSH, SW26 SW_PUSH, SW27 SW_PUSH, SW28 SW_PUSH, SW29 SW_PUSH, SW3 SW_PUSH, SW30 SW_PUSH, SW31 SW_PUSH, SW32 SW_PUSH, SW33 SW_PUSH, SW34 SW_PUSH, SW35 SW_PUSH, SW36 SW_PUSH, SW37 SW_PUSH, SW38 SW_PUSH, SW39 SW_PUSH, SW4 SW_PUSH, SW40 SW_PUSH, SW41 SW_PUSH, SW42 SW_PUSH, SW43 SW_PUSH, SW44 SW_PUSH, SW45 SW_PUSH, SW46 SW_PUSH, SW47 SW_PUSH, SW48 SW_PUSH, SW49 SW_PUSH, SW5 SW_PUSH, SW50 SW_PUSH, SW51 SW_PUSH, SW52 SW_PUSH, SW53 SW_PUSH, SW54 SW_PUSH, SW55 SW_PUSH, SW56 SW_PUSH, SW57 SW_PUSH, SW58 SW_PUSH, SW59 SW_PUSH, SW6 SW_PUSH, SW60 SW_PUSH, SW61 SW_PUSH, SW62 SW_PUSH, SW63 SW_PUSH, SW64 SW_PUSH, SW65 SW_PUSH, SW66 SW_PUSH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

Commit message: fix
Parts:
- removed L76: SK6812MINI, kbd_Parts:LED_SK6812MINI-E_BL, symbol Salicylic_kbd:LED_SK6812MINI-E
- removed SW76: SW_PUSH, kbd_SW:CherryMX_Hotswap_1u, symbol Switch:SW_Push
- added SW76: Rotary_Encoder_Switch, kbd_Parts:RotaryEncoder_EC12E, symbol Device:Rotary_Encoder_Switch
- renumbered L77 to L76
Connections:
- net Col7: now also SW76.S2
- net GND: now also SW76.C
- net A1: now reaches U1.11 (B4/PIN11)
- net A1: now also SW76.A
- net B1: now reaches U1.12 (B5/PIN12)
- net B1: now also SW76.B
- net at D76.1 (K): now also SW76.S1
- net at L76.3 (DIN): now also L75.1 (DOUT)
- net Reset: no longer names the net of U1.22 (RST)
- no-connect marks 6 -> 5
Other:
- moved on the sheet: L76
Changed lines of the file:
@@
 Text GLabel 1450 1725 0    50   Input ~ 0
 Row1
-Text GLabel 2850 1425 2    50   Input ~ 0
-Reset
 $Comp
 L power:PWR_FLAG #FLG01
@@
 NoConn ~ 1450 1325
 NoConn ~ 2850 2325
-NoConn ~ 1450 2225
-NoConn ~ 1450 2325
 Wire Wire Line
 	1450 1125 925  1125
@@
 $EndComp
 $Comp
-L power:GND #PWR022
+L power:GND #PWR023
 U 1 1 5CB45E4A
 P 13000 1400
-F 0 "#PWR022" H 13000 1150 50  0001 C CNN
+F 0 "#PWR023" H 13000 1150 50  0001 C CNN
 F 1 "GND" H 13005 1227 50  0000 C CNN
 F 2 "" H 13000 1400 50  0001 C CNN
@@
 Connection ~ 2350 6800
 Wire Wire Line
-	12425 3125 12425 3625
-Wire Wire Line
 	11775 3125 11775 3625
 Wire Wire Line
@@
 Col7
 $Comp
-L Switch:SW_Push SW76
-U 1 1 612B3E7E
-P 12625 3625
-F 0 "SW76" H 12625 3880 50  0000 C CNN
-F 1 "SW_PUSH" H 12625 3789 50  0000 C CNN
-F 2 "kbd_SW:CherryMX_Hotswap_1u" H 12625 3625 50  0001 C CNN
-F 3 "" H 12625 3625 50  0000 C CNN
-	1    12625 3625
-	1    0    0    -1
-$EndComp
-$Comp
 L Switch:SW_Push SW77
 U 1 1 612B3E5B
@@
 Wire Wire Line
 	10225 6800 10875 6800
-Connection ~ 12425 3625
 Wire Wire Line
 	10875 3925 11525 3925
@@
 	7300 12400 7300 13000
 $Comp
-L Salicylic_kbd:LED_SK6812MINI-E L76
-U 1 1 62E6D551
-P 8575 10600
-F 0 "L76" H 8575 10338 51  0000 C CNN
-F 1 "SK6812MINI" H 8575 10403 16  0000 C CNN
-F 2 "kbd_Parts:LED_SK6812MINI-E_BL" H 8575 10600 60  0001 C CNN
-F 3 "" H 8575 10600 60  0001 C CNN
-	1    8575 10600
-	0    1    1    0
-$EndComp
-$Comp
 L Salicylic_kbd:LED_SK6812MINI-E L73
 U 1 1 62E6D55B
@@
 Wire Wire Line
 	8875 9400 8875 10000
-Connection ~ 8875 10000
-Wire Wire Line
-	8875 10000 8875 10600
 Wire Wire Line
 	8275 7600 8275 8200
@@
 Wire Wire Line
 	8275 9400 8275 10000
-Connection ~ 8275 10000
-Wire Wire Line
-	8275 10000 8275 10600
 Wire Wire Line
 	1700 13300 2175 13300
@@
 Wire Wire Line
 	8075 7300 8575 7300
-Connection ~ 8875 10600
-Connection ~ 8275 10600
-Wire Wire Line
-	8875 10600 8875 11200
-Wire Wire Line
-	8275 10600 8275 11200
 $Comp
-L Salicylic_kbd:LED_SK6812MINI-E L77
+L Salicylic_kbd:LED_SK6812MINI-E L76
 U 1 1 62E6D547
-P 8575 11200
-F 0 "L77" H 8575 10938 51  0000 C CNN
-F 1 "SK6812MINI" H 8575 11003 16  0000 C CNN
-F 2 "kbd_Parts:LED_SK6812MINI-E_BL" H 8575 11200 60  0001 C CNN
-F 3 "" H 8575 11200 60  0001 C CNN
-	1    8575 11200
+P 8575 10600
+F 0 "L76" H 8575 10338 51  0000 C CNN
+F 1 "SK6812MINI" H 8575 10403 16  0000 C CNN
+F 2 "kbd_Parts:LED_SK6812MINI-E_BL" H 8575 10600 60  0001 C CNN
+F 3 "" H 8575 10600 60  0001 C CNN
+	1    8575 10600
 	0    1    1    0
 $EndComp
@@
 L power:GND #PWR020
 U 1 1 623C0DA7
-P 8275 11200
-F 0 "#PWR020" H 8275 10950 50  0001 C CNN
-F 1 "GND" H 8280 11027 50  0000 C CNN
-F 2 "" H 8275 11200 50  0001 C CNN
-F 3 "" H 8275 11200 50  0001 C CNN
-	1    8275 11200
-	1    0    0    -1
+P 8275 10600
+F 0 "#PWR020" H 8275 10350 50  0001 C CNN
+F 1 "GND" H 8280 10427 50  0000 C CNN
+F 2 "" H 8275 10600 50  0001 C CNN
+F 3 "" H 8275 10600 50  0001 C CNN
+	1    8275 10600
+	1    0    0    -1
+$EndComp
+NoConn ~ 8575 10900
+$Comp
+L Device:Rotary_Encoder_Switch SW76
+U 1 1 623823A9
+P 12625 3325
+F 0 "SW76" V 12579 3555 50  0000 L CNN
+F 1 "Rotary_Encoder_Switch" V 12670 3555 50  0000 L CNN
+F 2 "kbd_Parts:RotaryEncoder_EC12E" H 12475 3485 50  0001 C CNN
+F 3 "~" H 12625 3585 50  0001 C CNN
+	1    12625 3325
+	0    1    1    0
 $EndComp
-Connection ~ 8275 11200
+Wire Wire Line
+	12425 3125 12425 3625
+Wire Wire Line
+	12425 3625 12525 3625
+Connection ~ 12425 3625
 Wire Wire Line
 	12425 3625 12425 5825
-NoConn ~ 8575 11500
+Wire Wire Line
+	12725 3625 12825 3625
+$Comp
+L power:GND #PWR022
+U 1 1 624A227D
+P 12625 3025
+F 0 "#PWR022" H 12625 2775 50  0001 C CNN
+F 1 "GND" H 12630 2852 50  0000 C CNN
+F 2 "" H 12625 3025 50  0001 C CNN
+F 3 "" H 12625 3025 50  0001 C CNN
+	1    12625 3025
+	-1   0    0    1
+$EndComp
+Text GLabel 12725 3025 1    50   Input ~ 0
+A1
+Text GLabel 12525 3025 1    50   Input ~ 0
+B1
+Text GLabel 1450 2225 0    50   Input ~ 0
+A1
+Text GLabel 1450 2325 0    50   Input ~ 0
+B1
+NoConn ~ 2850 1425
+Wire Wire Line
+	8875 10000 8875 10600
+Connection ~ 8875 10000
+Wire Wire Line
+	8275 10000 8275 10600
+Connection ~ 8275 10000
+Connection ~ 8275 10600
 $EndSCHEMATC
