File: comfrey77_PCB/comfrey77.kicad_pcb (KiCad board)
At the start: 2 copper layers, 304.4 x 98.8 mm, 233 parts, among them J1 Conn_01x02, SW1 SW_PUSH, SW10 SW_PUSH, SW11 SW_PUSH, SW12 SW_PUSH, SW13 SW_PUSH, SW14 SW_PUSH, SW15 SW_PUSH, SW16 SW_PUSH, SW17 SW_PUSH, SW18 SW_PUSH, SW19 SW_PUSH, SW2 SW_PUSH, SW20 SW_PUSH, SW21 SW_PUSH, SW22 SW_PUSH, SW23 SW_PUSH, SW24 SW_PUSH, SW25 SW_PUSH, SW26 SW_PUSH, SW27 SW_PUSH, SW28 SW_PUSH, SW29 SW_PUSH, SW3 SW_PUSH, SW30 SW_PUSH, SW31 SW_PUSH, SW32 SW_PUSH, SW33 SW_PUSH, SW34 SW_PUSH, SW35 SW_PUSH, SW36 SW_PUSH, SW37 SW_PUSH, SW38 SW_PUSH, SW39 SW_PUSH, SW4 SW_PUSH, SW40 SW_PUSH, SW41 SW_PUSH, SW42 SW_PUSH, SW43 SW_PUSH, SW44 SW_PUSH, SW45 SW_PUSH, SW46 SW_PUSH, SW47 SW_PUSH, SW48 SW_PUSH, SW49 SW_PUSH, SW5 SW_PUSH, SW50 SW_PUSH, SW51 SW_PUSH, SW52 SW_PUSH, SW53 SW_PUSH, SW54 SW_PUSH, SW55 SW_PUSH, SW56 SW_PUSH, SW57 SW_PUSH, SW58 SW_PUSH, SW59 SW_PUSH, SW6 SW_PUSH, SW60 SW_PUSH, SW61 SW_PUSH, SW62 SW_PUSH, SW63 SW_PUSH, SW64 SW_PUSH, SW65 SW_PUSH, SW66 SW_PUSH, SW67 SW_PUSH, SW68 SW_PUSH, SW69 SW_PUSH, SW7 SW_PUSH, SW70 SW_PUSH, SW71 SW_PUSH, SW72 SW_PUSH, SW73 SW_PUSH, SW74 SW_PUSH, SW75 SW_PUSH, SW76 SW_PUSH, SW77 SW_PUSH, SW8 SW_PUSH, SW9 SW_PUSH, U1 BLEMicroPro

Commit message: fix
Parts:
- removed L77: SK6812MINI, kbd_Parts:LED_SK6812MINI-E_BL
- SW71: footprint kbd_SW:CherryMX_Hotswap_1u_Small1 -> kbd_SW:CherryMX_Hotswap_1u
- SW76: value SW_PUSH -> Rotary_Encoder_Switch; footprint kbd_SW:CherryMX_Hotswap_1u_Small1 -> kbd_Parts:RotaryEncoder_EC12E
- moved L57 21.4 mm to (104.8, 81.6)
- moved L37 21.4 mm to (181.0, 81.6)
- moved L47 21.4 mm to (142.9, 81.6)
- moved L67 21.4 mm to (66.7, 81.6)
- moved L58 21.4 mm to (95.2, 62.5)
- moved L38 21.4 mm to (171.4, 62.5)
- moved L48 21.4 mm to (133.3, 62.5)
- moved L70 21.4 mm to (47.6, 24.4)
- moved L50 21.4 mm to (123.8, 24.4)
- moved L60 21.4 mm to (85.7, 24.4)
- moved L40 21.4 mm to (161.9, 24.4)
- moved L68 21.4 mm to (57.1, 62.5)
- moved L76 21.3 mm to (28.6, 81.6)
- moved L35 21.2 mm to (190.5, 100.6)
- moved L45 21.2 mm to (152.4, 100.6)
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Connections:
- net Reset renamed Net-(U1-Pad22)
- U1 pad 11: Net-(U1-Pad11) -> A1
- U1 pad 12: Net-(U1-Pad12) -> B1
Routing:
- net Col2: track 488.1 -> 404.7 mm, vias 13 -> 14
- net Col4: track 458.0 -> 374.9 mm, vias 14 -> 18
- net GND: track 2074.5 -> 1995.1 mm, vias 155 -> 142
- net Col1: track 478.1 -> 418.3 mm, vias 15 -> 16
- net Col5: track 435.7 -> 376.5 mm
- net Col6: track 418.8 -> 364.1 mm, vias 10 -> 9
- net Row2: track 419.6 -> 369.6 mm
- net Col3: track 437.5 -> 393.0 mm, vias 15 -> 16
- net Net-(L56-Pad1): track 15.1 -> 46.4 mm, vias 0 -> 2
- net Row1: track 375.5 -> 344.2 mm, vias 0 -> 1
- net VCC: track 1651.8 -> 1621.3 mm
- net Col0: track 494.4 -> 466.6 mm
- net A1: track 0.00 -> 24.0 mm
- net Net-(L76-Pad1): track 23.3 -> 0.00 mm, vias 2 -> 0
- net Net-(L36-Pad1): track 14.5 -> 37.4 mm, vias 0 -> 2
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
Commit message: fix
Parts:
- added G***: LOGO, ロゴ:Comfrey77_LOGO, F.Cu at (26.2, 105.7)
- moved L1 0.45 mm to (295.3, 24.9)
- moved D71 0.37 mm to (286.6, 27.9)
- moved U1 0.30 mm to (289.9, 28.9)
- moved L10 0.22 mm to (276.2, 24.8)
Routing:
- net LED: track 36.3 -> 34.0 mm
- net Net-(L17-Pad1): track 27.7 -> 25.9 mm
- net Net-(L37-Pad1): track 25.5 -> 24.0 mm
- net Net-(L23-Pad1): track 28.8 -> 27.5 mm
- net Row0: track 352.1 -> 353.1 mm
- net Net-(L43-Pad1): track 28.5 -> 29.6 mm
- net Col0: track 466.6 -> 467.6 mm
- net Net-(L33-Pad1): track 28.8 -> 29.8 mm
- net Net-(L1-Pad1): track 27.3 -> 26.7 mm
- net Row2: track 369.6 -> 369.0 mm
- net VCC: track 1621.3 -> 1620.8 mm
- net Net-(L26-Pad1): track 36.8 -> 37.3 mm
